Commit message: apcar urdf fixed

File: models/vehicles/apcar/apcar.urdf (robot description, URDF)
Before this commit: robot apcar, 13 links, 12 joints
Links:
- link chassis: geometry collision mesh filename=package://apcar_ros_description/models/apcar_simplified.stl; visual mesh filename=package://apcar_ros_description/models/apcar_base.stl
- link steering_wheel: geometry collision cylinder length=0.04 radius=0.18; visual mesh filename=package://apcar_ros_description/models/steering_wheel.stl scale=0.007 0.007 0.007
- link wheel_back_left: geometry collision cylinder length=0.02 radius=0.24988162878124287; collision cylinder length=0.03 radius=0.24973358585766042
- link wheel_back_right: geometry collision cylinder length=0.02 radius=0.24988162878124287; collision cylinder length=0.03 radius=0.24973358585766042
- link wheel_front_left: geometry collision cylinder length=0.02 radius=0.24988162878124287; collision cylinder length=0.03 radius=0.24973358585766042
- link wheel_front_right: geometry collision cylinder length=0.02 radius=0.24988162878124287; collision cylinder length=0.03 radius=0.24973358585766042
Joints:
- joint axle_back_left: axis 0 0 -1 -> 0 0 1; origin xyz=0.02 0 0 rpy=0 1.5707963267948966 0 -> xyz=-0.02 0 0 rpy=0 1.5707963267948966 0
- joint axle_back_right: axis 0 0 -1 -> 0 0 1; origin xyz=-0.02 0 0 rpy=0 1.5707963267948966 0 -> xyz=0.02 0 0 rpy=0 1.5707963267948966 0
- joint axle_front_left: axis 0 0 -1 -> 0 0 1; origin xyz=0.02 0 0 rpy=0 1.5707963267948966 0 -> xyz=-0.02 0 0 rpy=0 1.5707963267948966 0
- joint axle_front_right: axis 0 0 -1 -> 0 0 1; origin xyz=-0.02 0 0 rpy=0 1.5707963267948966 0 -> xyz=0.02 0 0 rpy=0 1.5707963267948966 0
- joint base_link_to_chassis: origin xyz=0 0 0 -> xyz=0 0 0 rpy=0 0 0
- joint shock_absorber_back_left: origin xyz=      -0.4720000000000001      0.0      0.0      -> xyz=      0.0      0.4650000000000001      0.0      rpy=0 0 1.5707963267948966
- joint shock_absorber_back_right: origin xyz=      0.4720000000000001      0.0      0.0      -> xyz=      0.0      -0.4650000000000001      0.0      rpy=0 0 1.5707963267948966
- joint shock_absorber_front_left: origin xyz=      -0.4720000000000001      2.3      0.0      -> xyz=      2.3      0.4650000000000001      0.0      rpy=0 0 1.5707963267948966
- joint shock_absorber_front_right: origin xyz=      0.4720000000000001      2.3      0.0      -> xyz=      2.3      -0.4650000000000001      0.0      rpy=0 0 1.5707963267948966
- joint steering_wheel_to_chassis: origin xyz=-0.3 1.7 0.65 rpy=1.2217304763960306 0 0 -> xyz=1.7 0.3 0.65 rpy=1.2217304763960306 0 -1.5707963267948966

Commit message: apcar fix

File: models/vehicles/apcar/apcar.urdf (robot description, URDF)
Before this commit: robot apcar, 13 links, 12 joints
Links:
- link chassis: geometry collision mesh filename=meshes/apcar_simplified.stl; visual mesh filename=meshes/apcar_base.stl
- link steering_wheel: geometry collision cylinder length=0.04 radius=0.18; visual mesh filename=meshes/steering_wheel.stl scale=0.007 0.007 0.007
- link wheel_back_left: geometry collision cylinder length=0.02 radius=0.24988162878124287; collision cylinder length=0.03 radius=0.24973358585766042
- link wheel_back_right: geometry collision cylinder length=0.02 radius=0.24988162878124287; collision cylinder length=0.03 radius=0.24973358585766042
- link wheel_front_left: geometry collision cylinder length=0.02 radius=0.24988162878124287; collision cylinder length=0.03 radius=0.24973358585766042
- link wheel_front_right: geometry collision cylinder length=0.02 radius=0.24988162878124287; collision cylinder length=0.03 radius=0.24973358585766042
